Commit message: 修复官方SLAM链路并补充感知联调证据

File: ros2_ws/src/hazardwalker_platform/src/unitree_guide/unitree_ros/robots/a1_description/xacro/gazebo.xacro (robot description, xacro)
@@ -322,30 +322,33 @@
     <gazebo reference="laser_livox">
         <sensor type="ray" name="laser_livox">
-            <pose>0 0 0 0 0 0</pose>
+            <!-- laser_livox 链路俯仰约 +45°；反向补偿后 ray 扫描面保持水平。 -->
+            <pose>0 0 0 0 -0.785 0</pose>
             <visualize>true</visualize>
             <update_rate>10</update_rate>
+            <!-- ray 是 sensor 的 SDF 子元素，不能嵌在 ROS plugin 内；错误嵌套
+                 会退回 640 个全 inf、量程和角度均为 0 的无效默认扫描。 -->
+            <ray>
+                <scan>
+                    <horizontal>
+                        <samples>360</samples>
+                        <resolution>1</resolution>
+                        <min_angle>${-M_PI}</min_angle>
+                        <max_angle>${M_PI}</max_angle>
+                    </horizontal>
+                </scan>
+                <range>
+                    <min>0.1</min>
+                    <max>40.0</max>
+                    <resolution>0.01</resolution>
+                </range>
+                <noise>
+                    <type>gaussian</type>
+                    <mean>0.0</mean>
+                    <stddev>0.005</stddev>
+                </noise>
+            </ray>
             <plugin name="gazebo_ros_laser_controller" filename="libgazebo_ros_laser.so">
                 <topicName>/scan</topicName>
-                <frameName>laser_livox</frameName>
-                <ray>
-                    <scan>
-                        <horizontal>
-                            <samples>360</samples>
-                            <resolution>1</resolution>
-                            <min_angle>${-M_PI}</min_angle>
-                            <max_angle>${M_PI}</max_angle>
-                        </horizontal>
-                    </scan>
-                    <range>
-                        <min>0.1</min>
-                        <max>40.0</max>
-                        <resolution>0.01</resolution>
-                    </range>
-                    <noise>
-                        <type>gaussian</type>
-                        <mean>0.0</mean>
-                        <stddev>0.005</stddev>
-                    </noise>
-                </ray>
+                <frameName>laser_scan</frameName>
             </plugin>
         </sensor>

File: ros2_ws/src/hazardwalker_platform/src/unitree_guide/unitree_ros/robots/a1_description/xacro/robot.xacro (robot description, xacro)
@@ -132,4 +132,12 @@
         <child link="laser_livox"/>
     </joint>
+    <!-- Gazebo ray 经 -45° 补偿后实际是水平扫描；用独立水平帧表达这一
+         几何关系，避免 LaserScan 数据挂在上仰的 laser_livox 帧上污染 SLAM。 -->
+    <link name="laser_scan"/>
+    <joint name="laser_scan_joint" type="fixed">
+        <origin xyz="0.2 0 0.08" rpy="0 0 0"/>
+        <parent link="base"/>
+        <child link="laser_scan"/>
+    </joint>
     <!-- livox mid360-imu -->
     <!-- 对于本体 -->

Commit message: 负责人集成：固化房间巡检、感知闭环与仿真稳定启动

File: ros2_ws/src/hazardwalker_platform/src/unitree_guide/unitree_ros/robots/a1_description/xacro/gazebo.xacro (robot description, xacro)
@@ -318,6 +318,9 @@
         <kd  value="1.0"/>
     </gazebo>
-     <!-- gazebo livox mid360 plugins -->
+    <!-- gazebo livox mid360 plugins -->
     <xacro:property name="M_PI" value="3.14159"/>
+    <xacro:if value="$(arg ENABLE_LIDAR)">
+    <!-- 水平 360° 扫描独立服务 Cartographer/避障；三维 profile 额外启动
+         Mid-360，不能用稀疏三维切片覆盖 /scan。 -->
     <gazebo reference="laser_livox">
         <sensor type="ray" name="laser_livox">
@@ -354,4 +357,53 @@
         </sensor>
     </gazebo>
+    <xacro:if value="$(arg ENABLE_LIVOX_3D)">
+    <gazebo reference="laser_livox">
+        <sensor type="ray" name="laser_livox_3d">
+            <pose>0 0 0 0 0 0</pose>
+            <!-- 传感器必须主动更新；仅创建 ROS publisher 不会让 Gazebo
+                 默认关闭的 ray sensor 产生扫描回调。 -->
+            <always_on>true</always_on>
+            <visualize>false</visualize>
+            <update_rate>10</update_rate>
+            <plugin name="gazebo_livox_mid360_controller"
+                    filename="liblivox_laser_simulation.so">
+                <ray>
+                    <scan>
+                        <horizontal>
+                            <samples>100</samples>
+                            <resolution>1</resolution>
+                            <min_angle>0</min_angle>
+                            <max_angle>${2*M_PI}</max_angle>
+                        </horizontal>
+                        <vertical>
+                            <samples>360</samples>
+                            <resolution>1</resolution>
+                            <min_angle>${-3.22/180*M_PI}</min_angle>
+                            <max_angle>${56.22/180*M_PI}</max_angle>
+                        </vertical>
+                    </scan>
+                    <range>
+                        <min>0.1</min>
+                        <max>30.0</max>
+                        <resolution>0.02</resolution>
+                    </range>
+                    <noise>
+                        <type>gaussian</type>
+                        <mean>0.0</mean>
+                        <stddev>0.005</stddev>
+                    </noise>
+                </ray>
+                <!-- Mid-360 真机约 20 万点/秒。仿真保留约 1.2 万条射线/帧，
+                     让非重复扫描在室内平面上仍有足够重叠供 LIO 配准。 -->
+                <samples>24000</samples>
+                <downsample>2</downsample>
+                <repeat_pattern>true</repeat_pattern>
+                <csv_file_name>package://livox_laser_simulation/scan_mode/mid360.csv</csv_file_name>
+                <ros_topic>/livox/lidar_raw</ros_topic>
+            </plugin>
+        </sensor>
+    </gazebo>
+    </xacro:if>
+    </xacro:if>
     <!-- gazebo livox imu-link plugins -->
     <gazebo reference="livox_imu_link">

File: ros2_ws/src/hazardwalker_platform/src/unitree_guide/unitree_ros/robots/a1_description/xacro/robot.xacro (robot description, xacro)
@@ -2,4 +2,8 @@
 <robot name="a1" xmlns:xacro="http://www.ros.org/wiki/xacro">
     <xacro:arg name="DEBUG" default="false"/>
+    <!-- 默认关闭激光雷达，导航/SLAM profile 通过 ENABLE_LIDAR:=true 显式开启。 -->
+    <xacro:arg name="ENABLE_LIDAR" default="false"/>
+    <!-- 三维建图 profile 才启用真实 Mid-360 非重复扫描插件；默认二维保底。 -->
+    <xacro:arg name="ENABLE_LIVOX_3D" default="false"/>
     <xacro:include filename="$(find a1_description)/xacro/const.xacro"/>
     <xacro:include filename="$(find a1_description)/xacro/materials.xacro"/>
@@ -128,5 +132,9 @@
     <!-- 对于连接 -->
     <joint name="laser_livox_joint" type="fixed" >
-        <origin xyz="0.2 0 0.08" rpy="0 0.785 0" />
+        <!-- 负责人修复：原 z=0.08 只比 A1 机身顶部高约 2.3cm，水平
+             ray 会扫到髋腿并让 move_base 把机器人自身标成障碍。按真实
+             顶置 Mid-360 安装，并按 RL 动态步态的髋腿最高包络留足余量，
+             把扫描原点抬到 z=0.35。 -->
+        <origin xyz="0.2 0 0.35" rpy="0 0.785 0" />
         <parent link="base" />
         <child link="laser_livox"/>
@@ -136,5 +144,5 @@
     <link name="laser_scan"/>
     <joint name="laser_scan_joint" type="fixed">
-        <origin xyz="0.2 0 0.08" rpy="0 0 0"/>
+        <origin xyz="0.2 0 0.35" rpy="0 0 0"/>
         <parent link="base"/>
         <child link="laser_scan"/>

Commit message: 发布旧冻结版复用基线，整理构建运行入口与验证文档

File: ros2_ws/src/hazardwalker_platform/src/unitree_guide/unitree_ros/robots/a1_description/xacro/gazebo.xacro (robot description, xacro)
@@ -318,7 +318,9 @@
         <kd  value="1.0"/>
     </gazebo>
-     <!-- gazebo livox mid360 plugins -->
+    <!-- gazebo livox mid360 plugins -->
     <xacro:property name="M_PI" value="3.14159"/>
     <xacro:if value="$(arg ENABLE_LIDAR)">
+    <!-- 水平 360° 扫描独立服务 Cartographer/避障；三维 profile 额外启动
+         Mid-360，不能用稀疏三维切片覆盖 /scan。 -->
     <gazebo reference="laser_livox">
         <sensor type="ray" name="laser_livox">
@@ -355,4 +357,52 @@
         </sensor>
     </gazebo>
+    <xacro:if value="$(arg ENABLE_LIVOX_3D)">
+    <gazebo reference="laser_livox">
+        <sensor type="ray" name="laser_livox_3d">
+            <pose>0 0 0 0 0 0</pose>
+            <!-- 传感器必须主动更新；仅创建 ROS publisher 不会让 Gazebo
+                 默认关闭的 ray sensor 产生扫描回调。 -->
+            <always_on>true</always_on>
+            <visualize>false</visualize>
+            <update_rate>$(arg LIVOX_3D_UPDATE_RATE)</update_rate>
+            <plugin name="gazebo_livox_mid360_controller"
+                    filename="liblivox_laser_simulation.so">
+                <ray>
+                    <scan>
+                        <horizontal>
+                            <samples>100</samples>
+                            <resolution>1</resolution>
+                            <min_angle>0</min_angle>
+                            <max_angle>${2*M_PI}</max_angle>
+                        </horizontal>
+                        <vertical>
+                            <samples>360</samples>
+                            <resolution>1</resolution>
+                            <min_angle>${-3.22/180*M_PI}</min_angle>
+                            <max_angle>${56.22/180*M_PI}</max_angle>
+                        </vertical>
+                    </scan>
+                    <range>
+                        <min>0.1</min>
+                        <max>30.0</max>
+                        <resolution>0.02</resolution>
+                    </range>
+                    <noise>
+                        <type>gaussian</type>
+                        <mean>0.0</mean>
+                        <stddev>0.005</stddev>
+                    </noise>
+                </ray>
+                <!-- 独立展示默认约 600 点/秒；二维 SLAM/避障继续用 /scan。
+                     需要研究三维 LIO 时才显式提高，不能拖垮正式控制链。 -->
+                <samples>$(arg LIVOX_3D_SAMPLES)</samples>
+                <downsample>$(arg LIVOX_3D_DOWNSAMPLE)</downsample>
+                <repeat_pattern>true</repeat_pattern>
+                <csv_file_name>package://livox_laser_simulation/scan_mode/mid360.csv</csv_file_name>
+                <ros_topic>/livox/lidar_raw</ros_topic>
+            </plugin>
+        </sensor>
+    </gazebo>
+    </xacro:if>
     </xacro:if>
     <!-- gazebo livox imu-link plugins -->

File: ros2_ws/src/hazardwalker_platform/src/unitree_guide/unitree_ros/robots/a1_description/xacro/robot.xacro (robot description, xacro)
@@ -4,4 +4,10 @@
     <!-- 默认关闭激光雷达，导航/SLAM profile 通过 ENABLE_LIDAR:=true 显式开启。 -->
     <xacro:arg name="ENABLE_LIDAR" default="false"/>
+    <!-- 三维建图 profile 才启用真实 Mid-360 非重复扫描插件；默认二维保底。 -->
+    <xacro:arg name="ENABLE_LIVOX_3D" default="false"/>
+    <!-- 三维展示使用低负载采样；不得让传感器抢占控制器启动所需仿真步进。 -->
+    <xacro:arg name="LIVOX_3D_UPDATE_RATE" default="1"/>
+    <xacro:arg name="LIVOX_3D_SAMPLES" default="600"/>
+    <xacro:arg name="LIVOX_3D_DOWNSAMPLE" default="1"/>
     <xacro:include filename="$(find a1_description)/xacro/const.xacro"/>
     <xacro:include filename="$(find a1_description)/xacro/materials.xacro"/>
@@ -130,5 +136,9 @@
     <!-- 对于连接 -->
     <joint name="laser_livox_joint" type="fixed" >
-        <origin xyz="0.2 0 0.08" rpy="0 0.785 0" />
+        <!-- 负责人修复：原 z=0.08 只比 A1 机身顶部高约 2.3cm，水平
+             ray 会扫到髋腿并让 move_base 把机器人自身标成障碍。按真实
+             顶置 Mid-360 安装，并按 RL 动态步态的髋腿最高包络留足余量，
+             把扫描原点抬到 z=0.35。 -->
+        <origin xyz="0.2 0 0.35" rpy="0 0.785 0" />
         <parent link="base" />
         <child link="laser_livox"/>
@@ -138,5 +148,5 @@
     <link name="laser_scan"/>
     <joint name="laser_scan_joint" type="fixed">
-        <origin xyz="0.2 0 0.08" rpy="0 0 0"/>
+        <origin xyz="0.2 0 0.35" rpy="0 0 0"/>
         <parent link="base"/>
         <child link="laser_scan"/>
